Commit message: front leg done

File: body.urdf (robot description, URDF)
Before this commit: robot robot, 3 links, 2 joints
Links:
- link Frontleg: geometry collision box size=0.2 1 0.2; visual box size=0.2 1 0.2
Joints:
- joint Torso_Frontleg: origin xyz=-0.5 0 1 rpy=0 0 0 -> xyz=0 0.5 1 rpy=0 0 0

Commit message: backleg done

File: body.urdf (robot description, URDF)
Before this commit: robot robot, 3 links, 2 joints
Links:
- link Backleg: geometry collision box size=0.2 1 0.2; visual box size=0.2 1 0.2
Joints:
- joint Torso_Backleg: origin xyz=0.5 0 1 rpy=0 0 0 -> xyz=0 -0.5 1 rpy=0 0 0

Commit message: joint axis changed

File: body.urdf (robot description, URDF)
Before this commit: robot robot, 3 links, 2 joints
Joints:
- joint Torso_Backleg: axis 0 1 0 -> 1 0 0
- joint Torso_Frontleg: axis 0 1 0 -> 1 0 0

Commit message: leftleg done

File: body.urdf (robot description, URDF)
Before this commit: robot robot, 3 links, 2 joints
Links:
- added link Leftleg, mass 1; collision box size=1 0.2 0.2; visual box size=1 0.2 0.2
Joints:
- added joint Torso_Leftleg: type revolute, parent Torso, child Leftleg, origin xyz=-0.5 0 1 rpy=0 0 0, axis 1 0 0, limit lower=-3.14159 upper=3.14159 effort=0.0 velocity=0.0

Commit message: QUADSPIDER

File: body.urdf (robot description, URDF)
Before this commit: robot robot, 5 links, 4 joints
Links:
- removed link RightLeg
- added link LowerBackleg, mass 1; collision box size=0.2 0.2 1; visual box size=0.2 0.2 1
- added link LowerFrontleg, mass 1; collision box size=0.2 0.2 1; visual box size=0.2 0.2 1
- added link LowerLeftleg, mass 1; collision box size=0.2 0.2 1; visual box size=0.2 0.2 1
- added link LowerRightleg, mass 1; collision box size=0.2 0.2 1; visual box size=0.2 0.2 1
- added link Rightleg, mass 1; collision box size=1 0.2 0.2; visual box size=1 0.2 0.2
Joints:
- removed joint Torso_RightLeg
- added joint Backleg_LowerBackleg: type revolute, parent Backleg, child LowerBackleg, origin xyz=0 -1 0 rpy=0 0 0, axis 1 0 0, limit lower=-3.14159 upper=3.14159 effort=0.0 velocity=0.0
- added joint Frontleg_LowerFrontleg: type revolute, parent Frontleg, child LowerFrontleg, origin xyz=0 1 0 rpy=0 0 0, axis 1 0 0, limit lower=-3.14159 upper=3.14159 effort=0.0 velocity=0.0
- added joint Leftleg_LowerLeftleg: type revolute, parent Leftleg, child LowerLeftleg, origin xyz=-1 0 0 rpy=0 0 0, axis 1 0 0, limit lower=-3.14159 upper=3.14159 effort=0.0 velocity=0.0
- added joint Rightleg_LowerRightleg: type revolute, parent Rightleg, child LowerRightleg, origin xyz=1 0 0 rpy=0 0 0, axis 1 0 0, limit lower=-3.14159 upper=3.14159 effort=0.0 velocity=0.0
- added joint Torso_Rightleg: type revolute, parent Torso, child Rightleg, origin xyz=0.5 0 1 rpy=0 0 0, axis 1 0 0, limit lower=-3.14159 upper=3.14159 effort=0.0 velocity=0.0

Commit message: less buggy

File: body.urdf (robot description, URDF)
Before this commit: robot robot, 9 links, 8 joints
Joints:
- joint Leftleg_LowerLeftleg: axis 1 0 0 -> 0 1 0
- joint Rightleg_LowerRightleg: axis 1 0 0 -> 0 1hh 0
- joint Torso_Leftleg: axis 1 0 0 -> 0 1 0
- joint Torso_Rightleg: axis 1 0 0 -> 0 1 0
