Commit message: they can appear in a race like starting pos + constants added + cleanup

File: body0.urdf (robot description, URDF)
Before this commit: robot robot, 9 links, 8 joints
Joints:
- joint Torso_Backleg: origin xyz=0 -0.5 1 rpy=0 0 0 -> xyz=0 -2.5 1 rpy=0 0 0
- joint Torso_Frontleg: origin xyz=0 0.5 1 rpy=0 0 0 -> xyz=0 -1.5 1 rpy=0 0 0
- joint Torso_Leftleg: origin xyz=-0.5 0 1 rpy=0 0 0 -> xyz=-0.5 -2.0 1 rpy=0 0 0
- joint Torso_Rightleg: origin xyz=0.5 0 1 rpy=0 0 0 -> xyz=0.5 -2.0 1 rpy=0 0 0

File: body1.urdf (robot description, URDF)
Before this commit: robot robot, 9 links, 8 joints
Joints:
- joint Torso_Backleg: origin xyz=0 0.5 1 rpy=0 0 0 -> xyz=0 1.5 1 rpy=0 0 0
- joint Torso_Frontleg: origin xyz=0 1.5 1 rpy=0 0 0 -> xyz=0 2.5 1 rpy=0 0 0
- joint Torso_Leftleg: origin xyz=-0.5 1 1 rpy=0 0 0 -> xyz=-0.5 2.0 1 rpy=0 0 0
- joint Torso_Rightleg: origin xyz=0.5 1 1 rpy=0 0 0 -> xyz=0.5 2.0 1 rpy=0 0 0

Commit message: all robots move

File: body0.urdf (robot description, URDF)
Before this commit: robot robot, 9 links, 8 joints
Joints:
- joint Rightleg_LowerRightleg: axis 0 1hh 0 -> 0 1 0
- joint Torso_Backleg: origin xyz=0 -2.5 1 rpy=0 0 0 -> xyz=0 -10.5 1 rpy=0 0 0
- joint Torso_Frontleg: origin xyz=0 -1.5 1 rpy=0 0 0 -> xyz=0 -9.5 1 rpy=0 0 0
- joint Torso_Leftleg: origin xyz=-0.5 -2.0 1 rpy=0 0 0 -> xyz=-0.5 -10.0 1 rpy=0 0 0
- joint Torso_Rightleg: origin xyz=0.5 -2.0 1 rpy=0 0 0 -> xyz=0.5 -10.0 1 rpy=0 0 0

File: body2.urdf (robot description, URDF)
Before this commit: robot robot, 9 links, 8 joints
Joints:
- joint Torso_Backleg: origin xyz=0 -5.5 1 rpy=0 0 0 -> xyz=0 -0.5 1 rpy=0 0 0
- joint Torso_Frontleg: origin xyz=0 -4.5 1 rpy=0 0 0 -> xyz=0 0.5 1 rpy=0 0 0
- joint Torso_Leftleg: origin xyz=-0.5 -5.0 1 rpy=0 0 0 -> xyz=-0.5 0.0 1 rpy=0 0 0
- joint Torso_Rightleg: origin xyz=0.5 -5.0 1 rpy=0 0 0 -> xyz=0.5 0.0 1 rpy=0 0 0

File: body3.urdf (robot description, URDF)
Before this commit: robot robot, 9 links, 8 joints
Joints:
- joint Torso_Backleg: origin xyz=0 -5.5 1 rpy=0 0 0 -> xyz=0 4.5 1 rpy=0 0 0
- joint Torso_Frontleg: origin xyz=0 -4.5 1 rpy=0 0 0 -> xyz=0 5.5 1 rpy=0 0 0
- joint Torso_Leftleg: origin xyz=-0.5 -5.0 1 rpy=0 0 0 -> xyz=-0.5 5.0 1 rpy=0 0 0
- joint Torso_Rightleg: origin xyz=0.5 -5.0 1 rpy=0 0 0 -> xyz=0.5 5.0 1 rpy=0 0 0

File: body4.urdf (robot description, URDF)
Before this commit: robot robot, 9 links, 8 joints
Joints:
- joint Torso_Backleg: origin xyz=0 -5.5 1 rpy=0 0 0 -> xyz=0 9.5 1 rpy=0 0 0
- joint Torso_Frontleg: origin xyz=0 -4.5 1 rpy=0 0 0 -> xyz=0 10.5 1 rpy=0 0 0
- joint Torso_Leftleg: origin xyz=-0.5 -5.0 1 rpy=0 0 0 -> xyz=-0.5 10.0 1 rpy=0 0 0
- joint Torso_Rightleg: origin xyz=0.5 -5.0 1 rpy=0 0 0 -> xyz=0.5 10.0 1 rpy=0 0 0
